File: ECE411RFIDDoorLock/ESP8266/ESP8266 RFID Schematic.brd (EAGLE design)
At the start: 61 x 43.8 mm, 32 parts, among them J4 1050170001, M1 SERVO, Q3 MMBT2222ALT1GOSCT-ND, T1 600mA/40V, T2 600mA/40V, U1 CP2104, U2 AP2112K-3.3TRG1, X1 ESP-12E

Commit message: Revert
Parts:
- R11: value 10k -> 4.7k
Connections:
- removed net N$4: R9.1, X1.3
- net CH_PD: now also R9.1, X1.3
Routing:
- net GPIO5/SCL: track 62.1 -> 75.6 mm
- net CH_PD: track 71.7 -> 74.2 mm

Commit message: Fixes and updates
Routing:
- net RESET: track 62.1 -> 56.7 mm
